Commit message: [SmallApartment] fixed wrongly positioned link

File: resources/apartment-small.urdf (robot description, URDF)
Before this commit: robot apartment, 102 links, 101 joints
Joints:
- joint table_area_main_temp_raytest_fix_joint: origin xyz=5 4 0 rpy=0 0 1.57 -> xyz=5 4 0.705 rpy=0 0 1.57
