Commit message: continued working on lab demo

File: resources/robots/tracy.urdf (robot description, URDF)
Before this commit: robot tracy, 51 links, 50 joints
Links:
- link camera_link: geometry collision sphere radius=0.05; visual mesh filename=package://pycram/resources/objects/d435.dae scale=1.0 1.0 1.0
Joints:
- joint camera_link_joint: origin xyz=0.01 0.0 -0.026 rpy=0.0484812 1.25792843 0.057068 -> xyz=0.04 0.0 -0.026 rpy=2.75 0 1.57

Commit message: [labdemo] added petri dish and tracy now puts tray back into incubator

File: resources/robots/tracy.urdf (robot description, URDF)
Before this commit: robot tracy, 51 links, 50 joints
Joints:
- joint camera_link_joint: origin xyz=0.04 0.0 -0.026 rpy=2.75 0 1.57 -> xyz=0.04 0.0 -0.026 rpy=2.2 0 1.57
